Commit message: move laikago to laikago_description

File: laikago_description/robot/const.xacro (robot description, xacro)
@@ -1,4 +1,4 @@
 <?xml version="1.0"?>
-<robot name="laikago" xmlns:xacro="http://www.ros.org/wiki/xacro">
+<robot name="laikago_description" xmlns:xacro="http://www.ros.org/wiki/xacro">
     <!-- Constants for robot dimensions -->
     <xacro:property name="PI" value="3.1415926535897931"/>

File: laikago_description/robot/leg.xacro (robot description, xacro)
@@ -1,5 +1,5 @@
 <?xml version="1.0"?>
 <robot xmlns:xacro="http://www.ros.org/wiki/xacro">
-    <xacro:include filename="$(find laikago)/robot/transmission.xacro"/>
+    <xacro:include filename="$(find laikago_description)/robot/transmission.xacro"/>
     <xacro:macro name="leg" params="name mirror mirror_dae front_hind front_hind_dae *origin">
         <joint name="${name}_hip_joint" type="revolute">
@@ -31,5 +31,5 @@
                 </xacro:if>
                 <geometry>
-                    <mesh filename="package://laikago/meshes/hip.dae" scale="1 1 1"/>
+                    <mesh filename="package://laikago_description/meshes/hip.dae" scale="1 1 1"/>
                 </geometry>
                 <material name="orange"/>
@@ -77,8 +77,8 @@
                 <geometry>
                     <xacro:if value="${mirror_dae == 'true'}">
-                        <mesh filename="package://laikago/meshes/thigh.dae" scale="1 1 1"/>
+                        <mesh filename="package://laikago_description/meshes/thigh.dae" scale="1 1 1"/>
                     </xacro:if>
                     <xacro:if value="${mirror_dae == 'false'}">
-                        <mesh filename="package://laikago/meshes/thigh_mirror.dae" scale="1 1 1"/>
+                        <mesh filename="package://laikago_description/meshes/thigh_mirror.dae" scale="1 1 1"/>
                     </xacro:if>
                 </geometry>
@@ -112,5 +112,5 @@
                 <origin rpy="0 0 0" xyz="0 0 0"/>
                 <geometry>
-                    <mesh filename="package://laikago/meshes/calf.dae" scale="1 1 1"/>
+                    <mesh filename="package://laikago_description/meshes/calf.dae" scale="1 1 1"/>
                 </geometry>
                 <material name="orange"/>

File: laikago_description/robot/robot.xacro (robot description, xacro)
@@ -1,7 +1,7 @@
 <?xml version="1.0"?>
-<robot name="laikago" xmlns:xacro="http://www.ros.org/wiki/xacro">
-    <xacro:include filename="$(find laikago)/robot/const.xacro"/>
-    <xacro:include filename="$(find laikago)/robot/materials.xacro"/>
-    <xacro:include filename="$(find laikago)/robot/leg.xacro"/>
+<robot name="laikago_description" xmlns:xacro="http://www.ros.org/wiki/xacro">
+    <xacro:include filename="$(find laikago_description)/robot/const.xacro"/>
+    <xacro:include filename="$(find laikago_description)/robot/materials.xacro"/>
+    <xacro:include filename="$(find laikago_description)/robot/leg.xacro"/>
     <!-- Base footpoint Link -->
     <link name="base">
@@ -23,5 +23,5 @@
             <origin rpy="0 0 0" xyz="0 0 0"/>
             <geometry>
-                <mesh filename="package://laikago/meshes/trunk.dae" scale="1 1 1"/>
+                <mesh filename="package://laikago_description/meshes/trunk.dae" scale="1 1 1"/>
             </geometry>
             <material name="orange"/>

Commit message: remove folder laikago_rviz

File: laikago_description/robot/const.xacro (robot description, xacro)
@@ -3,4 +3,5 @@
     <!-- Constants for robot dimensions -->
     <xacro:property name="PI" value="3.1415926535897931"/>
+    <xacro:property name="stick_mass" value="0.00001"/>
     <!-- simplified collision value -->
     <xacro:property name="trunk_width" value="0.172"/>
@@ -16,4 +17,6 @@
     <xacro:property name="calf_height" value="0.016"/>
     <xacro:property name="foot_radius" value="0.0265"/>
+    <xacro:property name="stick_radius" value="0.01"/>
+    <xacro:property name="stick_length" value="0.2"/>
     <!-- kinematic value -->
     <xacro:property name="thigh_offset" value="0.037"/>

File: laikago_description/robot/leg.xacro (robot description, xacro)
@@ -131,10 +131,8 @@
             </inertial>
         </link>
-        <joint name="${name}_foot_fixed" type="revolute">
+        <joint name="${name}_foot_fixed" type="fixed">
             <origin rpy="0 0 0" xyz="0 0 ${-(calf_length)}"/>
             <parent link="${name}_calf"/>
             <child link="${name}_foot"/>
-            <axis xyz="0 0 1"/>
-            <limit effort="100.0" velocity="0.05" lower="-0.001" upper="0.001"/>
         </joint>
         <link name="${name}_foot">
@@ -146,5 +144,5 @@
                 <material name="orange"/>
             </visual>
-            <collision name="${name}_foot_collision">
+            <collision>
                 <origin rpy="0 0 0" xyz="0 0 0"/>
                 <geometry>

File: laikago_description/robot/robot.xacro (robot description, xacro)
@@ -4,5 +4,15 @@
     <xacro:include filename="$(find laikago_description)/robot/materials.xacro"/>
     <xacro:include filename="$(find laikago_description)/robot/leg.xacro"/>
-    <!-- Base footpoint Link -->
+    <!-- Rollover Protection mode will add an additional stick on the top, use "true" or "false" to switch it. -->
+    <xacro:property name="rolloverProtection" value="false"/>
+    <!-- Debug mode will hung up the robot, use "true" or "false" to switch it. -->
+    <xacro:if value="$(arg DEBUG)">
+        <link name="world"/>
+        <joint name="base_static_joint" type="fixed">
+            <origin rpy="0 0 0" xyz="0 0 0"/>
+            <parent link="world"/>
+            <child link="base"/>
+        </joint>
+    </xacro:if>
     <link name="base">
         <visual>
@@ -18,5 +28,4 @@
         <child link="trunk"/>
     </joint>
-    <!-- Base Link -->
     <link name="trunk">
         <visual>
@@ -42,4 +51,33 @@
         </inertial>
     </link>
+    <xacro:if value="${(rolloverProtection == 'true')}">
+        <joint name="stick_joint" type="fixed">
+            <parent link="trunk"/>
+            <child link="stick_link"/>
+            <origin rpy="0 0 0" xyz="${0.18} 0 ${stick_length/2.0+0.08}"/>
+        </joint>
+        <link name="stick_link">
+            <visual>
+                <geometry>
+                    <cylinder length="${stick_length}" radius="${stick_radius}"/>
+                </geometry>
+                <origin rpy="0 0 0" xyz="0 0 0"/>
+                <material name="white"/>
+            </visual>
+            <collision>
+                <geometry>
+                    <cylinder length="${stick_length}" radius="${stick_radius}"/>
+                </geometry>
+                <origin rpy="0 0 0" xyz="0 0 0"/>
+            </collision>
+            <inertial>
+                <mass value="${stick_mass}"/>
+                <inertia
+                    ixx="${stick_mass / 2.0 * (stick_radius*stick_radius)}" ixy="0.0" ixz="0.0"
+                    iyy="${stick_mass / 12.0 * (3*stick_radius*stick_radius + stick_length*stick_length)}" iyz="0.0"
+                    izz="${stick_mass / 12.0 * (3*stick_radius*stick_radius + stick_length*stick_length)}"/>
+            </inertial>
+        </link>
+    </xacro:if>
     <joint name="imu_joint" type="fixed">
         <parent link="trunk"/>
