Commit message: Update robot.xacro

File: laikago_description/xacro/robot.xacro (robot description, xacro)
@@ -106,14 +106,14 @@
         </collision>
     </link>
-    <xacro:leg name="FL" mirror="1" mirror_dae="true" front_hind="1" front_hind_dae="true">
+    <xacro:leg name="FR" mirror="-1" mirror_dae="False" front_hind="1" front_hind_dae="True">
+        <origin rpy="0 0 0" xyz="${leg_offset_x} ${-leg_offset_y} 0"/>
+    </xacro:leg>
+    <xacro:leg name="FL" mirror="1" mirror_dae="True" front_hind="1" front_hind_dae="True">
         <origin rpy="0 0 0" xyz="${leg_offset_x} ${leg_offset_y} 0"/>
     </xacro:leg>
-    <xacro:leg name="FR" mirror="-1" mirror_dae="false" front_hind="1" front_hind_dae="true">
-        <origin rpy="0 0 0" xyz="${leg_offset_x} ${-leg_offset_y} 0"/>
-    </xacro:leg>
-    <xacro:leg name="RR" mirror="-1" mirror_dae="false" front_hind="-1" front_hind_dae="false">
+    <xacro:leg name="RR" mirror="-1" mirror_dae="False" front_hind="-1" front_hind_dae="False">
         <origin rpy="0 0 0" xyz="${-leg_offset_x} ${-leg_offset_y} 0"/>
     </xacro:leg>
-    <xacro:leg name="RL" mirror="1" mirror_dae="true" front_hind="-1" front_hind_dae="false">
+    <xacro:leg name="RL" mirror="1" mirror_dae="True" front_hind="-1" front_hind_dae="False">
         <origin rpy="0 0 0" xyz="${-leg_offset_x} ${leg_offset_y} 0"/>
     </xacro:leg>
